Commit message: initial push

File: urdf/alm_t1.urdf (robot description, URDF)
Before this commit: robot my_robo, 5 links, 4 joints
Links:
- added link vive_tracker_link; visual box size=0.1 0.1 0.1
Joints:
- added joint vive_tracker_joint: type fixed, parent base_link, child vive_tracker_link, origin xyz=-0.2 0 0.15 rpy=0 0 0

Commit message: fix .launch

File: urdf/alm_t1.urdf (robot description, URDF)
Before this commit: robot my_robo, 5 links, 4 joints
Joints:
- joint slider0_joint: origin xyz=0 0 -0.010 rpy=0 0 0 -> xyz=0.150 0 -0.010 rpy=0 0 0; type prismatic -> fixed
- joint slider1_joint: origin xyz=-0 0 -0.010 rpy=0 0 0 -> xyz=-0.150 0 -0.010 rpy=0 0 0; type prismatic -> fixed

Commit message: add tube arm

File: urdf/alm_t1.urdf (robot description, URDF)
Before this commit: robot my_robo, 6 links, 5 joints
Links:
- added link tubeL_link0; visual box size=0.12 0.02 0.02
- added link tubeL_link1; visual cylinder length=0.08 radius=0.02
- added link tubeR_link0; visual box size=0.12 0.02 0.02
- added link tubeR_link1; visual cylinder length=0.08 radius=0.02
Joints:
- added joint tubeL_joint0: type revolute, parent base_link, child tubeL_link0, origin xyz=-0.13 0.09 0.1 rpy=0 0 0, axis 0 0 1, limit lower=-1 upper=1 effort=1.0 velocity=1.0
- added joint tubeL_joint1: type fixed, parent tubeL_link0, child tubeL_link1, origin xyz=-0.12 0 -0.03 rpy=0 0 0
- added joint tubeR_joint0: type revolute, parent base_link, child tubeR_link0, origin xyz=-0.13 -0.09 0.1 rpy=0 0 0, axis 0 0 1, limit lower=-1 upper=1 effort=1.0 velocity=1.0
- added joint tubeR_joint1: type fixed, parent tubeR_link0, child tubeR_link1, origin xyz=-0.12 0 -0.03 rpy=0 0 0

Commit message: add tf bl rot pos

File: urdf/alm_t1.urdf (robot description, URDF)
Before this commit: robot my_robo, 10 links, 9 joints
Joints:
- joint tubeL_joint0: origin xyz=-0.13 0.09 0.1 rpy=0 0 0 -> xyz=-0.12580 0.0750 0.1 rpy=0 0 0
- joint tubeR_joint0: origin xyz=-0.13 -0.09 0.1 rpy=0 0 0 -> xyz=-0.12580 -0.0750 0.1 rpy=0 0 0

Commit message: modify a bug

File: urdf/alm_t1.urdf (robot description, URDF)
Before this commit: robot my_robo, 10 links, 9 joints
Joints:
- joint tubeL_joint1: origin xyz=-0.12 0 -0.03 rpy=0 0 0 -> xyz=-0.105 0 -0.03 rpy=0 0 0
- joint tubeR_joint1: origin xyz=-0.12 0 -0.03 rpy=0 0 0 -> xyz=-0.105 0 -0.03 rpy=0 0 0

Commit message: modify
viveの座標系を解決した

File: urdf/alm_t1.urdf (robot description, URDF)
Before this commit: robot my_robo, 10 links, 9 joints
Links:
- link tubeL_link1: geometry visual cylinder length=1.08 radius=0.02

Commit message: add br operation
brのノズルの制御も完成

File: urdf/alm_t1.urdf (robot description, URDF)
Before this commit: robot my_robo, 10 links, 9 joints
Links:
- link tubeR_link1: geometry visual cylinder length=1.08 radius=0.02
